File: HotKeyBoard.kicad_pcb (KiCad board)
At the start: 2 copper layers, 288.3 x 133.3 mm, 218 parts, among them J1 Conn_01x12_Socket, J2 Conn_01x12_Socket, SW1 SW_Push, SW10 SW_Push, SW11 SW_Push, SW12 SW_Push, SW13 SW_Push, SW14 SW_Push, SW15 SW_Push, SW16 SW_Push, SW17 SW_Push, SW18 SW_Push, SW19 SW_Push, SW2 SW_Push, SW20 SW_Push, SW21 SW_Push, SW22 SW_Push, SW23 SW_Push, SW24 SW_Push, SW25 SW_Push, SW26 SW_Push, SW27 SW_Push, SW28 SW_Push, SW29 SW_Push, SW3 SW_Push, SW30 SW_Push, SW31 SW_Push, SW32 SW_Push, SW33 SW_Push, SW34 SW_Push, SW35 SW_Push, SW36 SW_Push, SW37 SW_Push, SW38 SW_Push, SW39 SW_Push, SW4 SW_Push, SW40 SW_Push, SW41 SW_Push, SW42 SW_Push, SW43 SW_Push, SW44 SW_Push, SW45 SW_Push, SW46 SW_Push, SW47 SW_Push, SW48 SW_Push, SW49 SW_Push, SW5 SW_Push, SW50 SW_Push, SW51 SW_Push, SW52 SW_Push, SW53 SW_Push, SW54 SW_Push, SW55 SW_Push, SW56 SW_Push, SW57 SW_Push, SW58 SW_Push, SW59 SW_Push, SW6 SW_Push, SW60 SW_Push, SW61 SW_Push, SW62 SW_Push, SW63 SW_Push, SW64 SW_Push, SW65 SW_Push, SW66 SW_Push, SW67 SW_Push, SW68 SW_Push, SW69 SW_Push, SW7 SW_Push, SW70 SW_Push, SW71 SW_Push, SW72 SW_Push, SW8 SW_Push, SW9 SW_Push

Commit message: Moved function key
Parts:
- SW53, SW54, SW55, SW56: footprint Button_Switch_Keyboard:SW_Cherry_MX_1.25u_PCB -> Button_Switch_Keyboard:SW_Cherry_MX_1.00u_PCB
- SW69: footprint Button_Switch_Keyboard:SW_Cherry_MX_2.75u_PCB -> Button_Switch_Keyboard:SW_Cherry_MX_1.75u_PCB
- moved D58 230.7 mm to (409.3, 163.4), turned to 180 degrees
- moved D117 230.3 mm to (410.1, 179.5), turned to 180 degrees
- moved SW57 230.2 mm to (407.4, 166.4)
- moved D59 205.6 mm to (409.2, 144.4)
- moved SW58 205.2 mm to (407.4, 147.3)
- moved D118 201.7 mm to (406.0, 160.7), turned to 180 degrees
- moved SW59 38.1 mm to (197.8, 71.1)
- moved D119 38.0 mm to (200.3, 84.5)
- moved D60 37.7 mm to (199.7, 68.1)
- moved D116 16.8 mm to (390.7, 179.6), turned to 180 degrees
- moved SW56 16.7 mm to (388.3, 166.4)
- moved D57 16.6 mm to (389.7, 163.3)
- moved D115 12.1 mm to (371.6, 179.6)
- moved SW55 11.9 mm to (369.3, 166.4)
- moved D56 11.5 mm to (370.9, 163.3)
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Connections:
- J2 pad 10: 5V -> unconnected-(J2-Pin_10-Pad10)
Routing:
- net Col9: track 330.6 -> 279.2 mm, vias 6 -> 5
- net Pin11: track 501.3 -> 518.5 mm, vias 14 -> 12
- net Col6: track 322.8 -> 338.8 mm, vias 7 -> 9
- net Col8: track 267.9 -> 254.4 mm
- net Col10: track 287.0 -> 275.0 mm, vias 4 -> 5
- net Net-(D141-K): track 17.0 -> 28.1 mm
- net Col7: track 281.1 -> 289.2 mm, vias 2 -> 4
- net GND: track 62.0 -> 66.3 mm, vias 2 -> 3
- net Col11: track 310.7 -> 313.1 mm
- net Col12: track 396.6 -> 394.2 mm
- net Col5: track 344.4 -> 342.1 mm
- net Col4: track 304.4 -> 302.0 mm
- net Net-(D117-K): track 17.0 -> 18.8 mm
- net Net-(D116-K): track 17.0 -> 17.8 mm
- net Col3: track 296.3 -> 297.1 mm

Commit message: Changed to 75 layout without function row, but added makro column instead
Parts:
- moved D133 213.0 mm to (124.0, 122.6)
- moved SW61 213.0 mm to (121.6, 109.2)
- moved D62 212.7 mm to (123.0, 106.0)
- moved D49 116.2 mm to (427.8, 87.0)
- moved D120 115.9 mm to (428.8, 103.5)
- moved SW60 115.9 mm to (426.4, 90.2)
- moved D84 97.5 mm to (124.3, 179.7)
- moved D144 97.3 mm to (429.1, 179.7)
- moved SW24 97.1 mm to (121.6, 166.4)
- moved SW72 97.1 mm to (426.4, 166.4)
- moved D13 97.0 mm to (123.0, 163.2)
- moved D61 97.0 mm to (427.8, 163.2)
- moved D119 96.0 mm to (123.3, 141.6)
- moved D60 95.6 mm to (123.0, 125.1)
- moved D131 95.4 mm to (124.0, 160.7)
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Routing:
- net Col12: track 394.2 -> 593.0 mm, vias 7 -> 9
- net Col11: track 313.1 -> 511.8 mm, vias 6 -> 9
- net Pin7: track 462.4 -> 536.0 mm, vias 15 -> 12
- net Col5: track 342.1 -> 405.7 mm, vias 6 -> 10
- net Col9: track 279.2 -> 261.2 mm
- net Pin12: track 397.8 -> 413.1 mm, vias 16 -> 15
- net GND: track 66.3 -> 81.6 mm
- net Pin8: track 265.6 -> 250.9 mm
- net Pin11: track 518.5 -> 530.0 mm, vias 12 -> 14
- net Col2: track 291.3 -> 300.9 mm
- net Net-(D141-K): track 28.1 -> 18.7 mm
- net Col8: track 254.4 -> 263.1 mm, vias 4 -> 6
- net Col10: track 275.0 -> 283.2 mm, vias 5 -> 8
- net Col7: track 289.2 -> 295.7 mm, vias 4 -> 7
- net Col4: track 302.0 -> 305.1 mm, vias 5 -> 6
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Other:
- board size 288.3 x 133.3 mm -> 326.4 x 132.1 mm

Commit message: Added mounting holes
Parts:
- added H1: MountingHole, MountingHole:MountingHole_3.2mm_M3_DIN965, F.Cu at (118.4, 94.6)
- added H2: MountingHole, MountingHole:MountingHole_3.2mm_M3_DIN965, F.Cu at (412.6, 133.5)
- added H3: MountingHole, MountingHole:MountingHole_3.2mm_M3_DIN965, F.Cu at (298.8, 171.6)
- added H4: MountingHole, MountingHole:MountingHole_3.2mm_M3_DIN965, F.Cu at (220.0, 171.6)
Routing:
- net Col7: track 295.7 -> 292.6 mm
Changed lines of the file:
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@@
   (setup
     (pad_to_mask_clearance 0)
-    (grid_origin 414.3375 85.725)
+    (grid_origin 222.5675 171.577)
     (pcbplotparams
       (layerselection 0x00010fc_ffffffff)
@@
     )
   )
+  (footprint "MountingHole:MountingHole_3.2mm_M3_DIN965" (layer "F.Cu")
+    (at 118.4275 94.615)
+    (descr "Mounting Hole 3.2mm, no annular, M3, DIN965")
+    (tags "mounting hole 3.2mm no annular m3 din965")
+    (property "Sheetfile" "HotKeyBoard.kicad_sch")
+    (property "Sheetname" "")
+    (property "ki_description" "Mounting Hole without connection")
+    (property "ki_keywords" "mounting hole")
+    (attr exclude_from_pos_files)
+    (fp_text reference "H1" (at 0 -3.8) (layer "F.SilkS")
+        (effects (font (size 1 1) (thickness 0.15)))
+    )
+    (fp_text value "MountingHole" (at 0 3.8) (layer "F.Fab")
+        (effects (font (size 1 1) (thickness 0.15)))
+    )
+    (fp_text user "${REFERENCE}" (at 0 0) (layer "F.Fab")
+        (effects (font (size 1 1) (thickness 0.15)))
+    )
+    (fp_circle (center 0 0) (end 2.8 0)
+      (stroke (width 0.15) (type solid)) (fill none) (layer "Cmts.User"))
+    (fp_circle (center 0 0) (end 3.05 0)
+      (stroke (width 0.05) (type solid)) (fill none) (layer "F.CrtYd"))
+    (pad "" np_thru_hole circle (at 0 0) (size 3.2 3.2) (drill 3.2) (layers "*.Cu" "*.Mask"))
+  )
   (footprint "Button_Switch_Keyboard:SW_Cherry_MX_1.00u_PCB" (layer "F.Cu")
     (at 250.19 128.27)
@@
     )
   )
+  (footprint "MountingHole:MountingHole_3.2mm_M3_DIN965" (layer "F.Cu")
+    (at 298.7675 171.577)
+    (descr "Mounting Hole 3.2mm, no annular, M3, DIN965")
+    (tags "mounting hole 3.2mm no annular m3 din965")
+    (property "Sheetfile" "HotKeyBoard.kicad_sch")
+    (property "Sheetname" "")
+    (property "ki_description" "Mounting Hole without connection")
+    (property "ki_keywords" "mounting hole")
+    (attr exclude_from_pos_files)
+    (fp_text reference "H3" (at 0 -3.8) (layer "F.SilkS")
+        (effects (font (size 1 1) (thickness 0.15)))
+    )
+    (fp_text value "MountingHole" (at 0 3.8) (layer "F.Fab")
+        (effects (font (size 1 1) (thickness 0.15)))
+    )
+    (fp_text user "${REFERENCE}" (at 0 0) (layer "F.Fab")
+        (effects (font (size 1 1) (thickness 0.15)))
+    )
+    (fp_circle (center 0 0) (end 2.8 0)
+      (stroke (width 0.15) (type solid)) (fill none) (layer "Cmts.User"))
+    (fp_circle (center 0 0) (end 3.05 0)
+      (stroke (width 0.05) (type solid)) (fill none) (layer "F.CrtYd"))
+    (pad "" np_thru_hole circle (at 0 0) (size 3.2 3.2) (drill 3.2) (layers "*.Cu" "*.Mask"))
+  )
   (footprint "Diode_SMD:D_SOD-323" (layer "F.Cu")
     (at 155.060398 160.555398)
@@
     )
   )
+  (footprint "MountingHole:MountingHole_3.2mm_M3_DIN965" (layer "F.Cu")
+    (at 412.5595 133.477)
+    (descr "Mounting Hole 3.2mm, no annular, M3, DIN965")
+    (tags "mounting hole 3.2mm no annular m3 din965")
+    (property "Sheetfile" "HotKeyBoard.kicad_sch")
+    (property "Sheetname" "")
+    (property "ki_description" "Mounting Hole without connection")
+    (property "ki_keywords" "mounting hole")
+    (attr exclude_from_pos_files)
+    (fp_text reference "H2" (at 0 -3.8) (layer "F.SilkS")
+        (effects (font (size 1 1) (thickness 0.15)))
+    )
+    (fp_text value "MountingHole" (at 0 3.8) (layer "F.Fab")
+        (effects (font (size 1 1) (thickness 0.15)))
+    )
+    (fp_text user "${REFERENCE}" (at 0 0) (layer "F.Fab")
+        (effects (font (size 1 1) (thickness 0.15)))
+    )
+    (fp_circle (center 0 0) (end 2.8 0)
+      (stroke (width 0.15) (type solid)) (fill none) (layer "Cmts.User"))
+    (fp_circle (center 0 0) (end 3.05 0)
+      (stroke (width 0.05) (type solid)) (fill none) (layer "F.CrtYd"))
+    (pad "" np_thru_hole circle (at 0 0) (size 3.2 3.2) (drill 3.2) (layers "*.Cu" "*.Mask"))
+  )
   (footprint "Diode_SMD:D_SOD-323" (layer "F.Cu")
     (at 403.980398 106.199398)
@@
     )
   )
+  (footprint "MountingHole:MountingHole_3.2mm_M3_DIN965" (layer "F.Cu")
+    (at 220.0275 171.577)
+    (descr "Mounting Hole 3.2mm, no annular, M3, DIN965")
+    (tags "mounting hole 3.2mm no annular m3 din965")
+    (property "Sheetfile" "HotKeyBoard.kicad_sch")
+    (property "Sheetname" "")
+    (property "ki_description" "Mounting Hole without connection")
+    (property "ki_keywords" "mounting hole")
+    (attr exclude_from_pos_files)
+    (fp_text reference "H4" (at 0 -3.8) (layer "F.SilkS")
+        (effects (font (size 1 1) (thickness 0.15)))
+    )
+    (fp_text value "MountingHole" (at 0 3.8) (layer "F.Fab")
+        (effects (font (size 1 1) (thickness 0.15)))
+    )
+    (fp_text user "${REFERENCE}" (at 0 0) (layer "F.Fab")
+        (effects (font (size 1 1) (thickness 0.15)))
+    )
+    (fp_circle (center 0 0) (end 2.8 0)
+      (stroke (width 0.15) (type solid)) (fill none) (layer "Cmts.User"))
+    (fp_circle (center 0 0) (end 3.05 0)
+      (stroke (width 0.05) (type solid)) (fill none) (layer "F.CrtYd"))
+    (pad "" np_thru_hole circle (at 0 0) (size 3.2 3.2) (drill 3.2) (layers "*.Cu" "*.Mask"))
+  )
   (footprint "Diode_SMD:D_SOD-323" (layer "F.Cu")
     (at 303.972398 106.199398)
@@
   (segment (start 402.4375 134.023) (end 401.8915 133.477) (width 0.25) (layer "F.Cu") (net 18))
   (segment (start 374.76375 156.28675) (end 375.7295 155.321) (width 0.25) (layer "F.Cu") (net 18))
+  (segment (start 304.1015 165.2905) (end 299.366398 160.555398) (width 0.25) (layer "F.Cu") (net 18))
   (segment (start 299.366398 160.555398) (end 292.9 154.089) (width 0.25) (layer "F.Cu") (net 18))
   (segment (start 289.248398 142.055398) (end 283.375 136.182) (width 0.25) (layer "F.Cu") (net 18))
@@
   (segment (start 275.3175 101.2005) (end 275.3175 90.870255) (width 0.25) (layer "F.Cu") (net 18))
   (segment (start 275.4275 70.965) (end 275.4275 67.917) (width 0.25) (layer "F.Cu") (net 18))
-  (segment (start 299.112398 160.809398) (end 299.366398 160.555398) (width 0.25) (layer "F.Cu") (net 18))
+  (segment (start 304.1015 176.303398) (end 304.1015 165.2905) (width 0.25) (layer "F.Cu") (net 18))
   (segment (start 291.780398 141.505398) (end 291.230398 142.055398) (width 0.25) (layer "F.Cu") (net 18))
   (segment (start 277.9395 122.555) (end 277.9395 113.013255) (width 0.25) (layer "F.Cu") (net 18))
@@
   (segment (start 292.9 154.089) (end 292.9 142.625) (width 0.25) (layer "F.Cu") (net 18))
   (segment (start 278.6025 112.350255) (end 278.6025 104.4855) (width 0.25) (layer "F.Cu") (net 18))
-  (segment (start 299.112398 176.303398) (end 299.112398 160.809398) (width 0.25) (layer "F.Cu") (net 18))
   (segment (start 401.8915 131.958006) (end 406.7125 127.137006) (width 0.25) (layer "F.Cu") (net 18))
   (segment (start 401.8915 133.477) (end 401.8915 131.958006) (width 0.25) (layer "F.Cu") (net 18))
@@
   (via (at 283.5275 122.555) (size 0.8) (drill 0.4) (layers "F.Cu" "B.Cu") (free) (net 18))
   (via (at 277.9395 122.555) (size 0.8) (drill 0.4) (layers "F.Cu" "B.Cu") (free) (net 18))
-  (via (at 299.112398 176.303398) (size 0.8) (drill 0.4) (layers "F.Cu" "B.Cu") (free) (net 18))
+  (via (at 304.1015 176.303398) (size 0.8) (drill 0.4) (layers "F.Cu" "B.Cu") (free) (net 18))
   (via (at 375.7295 155.321) (size 0.8) (drill 0.4) (layers "F.Cu" "B.Cu") (net 18))
   (via (at 402.1455 154.813) (size 0.8) (drill 0.4) (layers "F.Cu" "B.Cu") (net 18))
   (segment (start 401.6375 155.321) (end 402.1455 154.813) (width 0.25) (layer "B.Cu") (net 18))
+  (segment (start 371.057898 176.303398) (end 374.2055 179.451) (width 0.25) (layer "B.Cu") (net 18))
   (segment (start 278.7015 67.691) (end 279.7175 66.675) (width 0.25) (layer "B.Cu") (net 18))
-  (segment (start 299.112398 176.303398) (end 371.057898 176.303398) (width 0.25) (layer "B.Cu") (net 18))
   (segment (start 375.7295 155.321) (end 401.6375 155.321) (width 0.25) (layer "B.Cu") (net 18))
-  (segment (start 371.057898 176.303398) (end 374.2055 179.451) (width 0.25) (layer "B.Cu") (net 18))
+  (segment (start 304.1015 176.303398) (end 371.057898 176.303398) (width 0.25) (layer "B.Cu") (net 18))
   (segment (start 275.6535 67.691) (end 278.7015 67.691) (width 0.25) (layer "B.Cu") (net 18))
   (segment (start 283.5275 122.555) (end 277.9395 122.555) (width 0.25) (layer "B.Cu") (net 18))
