File: HotKeyBoard.kicad_pcb (KiCad board)
At the start: 2 copper layers, 326.4 x 132.1 mm, 222 parts, among them J1 Conn_01x12_Socket, J2 Conn_01x12_Socket, SW1 SW_Push, SW10 SW_Push, SW11 SW_Push, SW12 SW_Push, SW13 SW_Push, SW14 SW_Push, SW15 SW_Push, SW16 SW_Push, SW17 SW_Push, SW18 SW_Push, SW19 SW_Push, SW2 SW_Push, SW20 SW_Push, SW21 SW_Push, SW22 SW_Push, SW23 SW_Push, SW24 SW_Push, SW25 SW_Push, SW26 SW_Push, SW27 SW_Push, SW28 SW_Push, SW29 SW_Push, SW3 SW_Push, SW30 SW_Push, SW31 SW_Push, SW32 SW_Push, SW33 SW_Push, SW34 SW_Push, SW35 SW_Push, SW36 SW_Push, SW37 SW_Push, SW38 SW_Push, SW39 SW_Push, SW4 SW_Push, SW40 SW_Push, SW41 SW_Push, SW42 SW_Push, SW43 SW_Push, SW44 SW_Push, SW45 SW_Push, SW46 SW_Push, SW47 SW_Push, SW48 SW_Push, SW49 SW_Push, SW5 SW_Push, SW50 SW_Push, SW51 SW_Push, SW52 SW_Push, SW53 SW_Push, SW54 SW_Push, SW55 SW_Push, SW56 SW_Push, SW57 SW_Push, SW58 SW_Push, SW59 SW_Push, SW6 SW_Push, SW60 SW_Push, SW61 SW_Push, SW62 SW_Push, SW63 SW_Push, SW64 SW_Push, SW65 SW_Push, SW66 SW_Push, SW67 SW_Push, SW68 SW_Push, SW69 SW_Push, SW7 SW_Push, SW70 SW_Push, SW71 SW_Push, SW72 SW_Push, SW8 SW_Push, SW9 SW_Push

Commit message: Fixed bug in keyboard matrix
Parts:
- removed D100, D101, D102, D103, D104, D105, D106, D107, D108, D109, D110, D111, D112, D113, D114, D115, D116, D117, D118, D119, D120, D121, D122, D123, D124, D125, D126, D127, D128, D129, D130, D131, D132, D133, D134, D135, D136, D137, D138, D139, D140, D141, D142, D143, D144, D73, D74, D75, D76, D77, D78, D79, D80, D81, D82, D83, D84, D85, D86, D87, D88, D89, D90, D91, D92, D93, D94, D95, D96, D97, D98, D99: D, Diode_SMD:D_SOD-323
- SW11, SW17, SW5: footprint Button_Switch_Keyboard:SW_Cherry_MX_1.00u_PCB -> Button_Switch_Keyboard:SW_Cherry_MX_1.25u_PCB
- SW12: footprint Button_Switch_Keyboard:SW_Cherry_MX_1.00u_PCB -> Button_Switch_Keyboard:SW_Cherry_MX_2.00u_PCB
- SW2, SW24: footprint Button_Switch_Keyboard:SW_Cherry_MX_1.00u_PCB -> Button_Switch_Keyboard:SW_Cherry_MX_1.50u_PCB
- SW23, SW4: footprint Button_Switch_Keyboard:SW_Cherry_MX_1.00u_PCB -> Button_Switch_Keyboard:SW_Cherry_MX_2.25u_PCB
- SW3, SW70: footprint Button_Switch_Keyboard:SW_Cherry_MX_1.00u_PCB -> Button_Switch_Keyboard:SW_Cherry_MX_1.75u_PCB
- SW35: footprint Button_Switch_Keyboard:SW_Cherry_MX_1.00u_PCB -> Button_Switch_Keyboard:SW_Cherry_MX_6.25u_PCB
- SW49, SW50, SW51: footprint Button_Switch_Keyboard:SW_Cherry_MX_1.25u_PCB -> Button_Switch_Keyboard:SW_Cherry_MX_1.00u_PCB
- SW52: footprint Button_Switch_Keyboard:SW_Cherry_MX_6.25u_PCB -> Button_Switch_Keyboard:SW_Cherry_MX_1.00u_PCB
- SW62, SW67: footprint Button_Switch_Keyboard:SW_Cherry_MX_1.50u_PCB -> Button_Switch_Keyboard:SW_Cherry_MX_1.00u_PCB
- SW63, SW69: footprint Button_Switch_Keyboard:SW_Cherry_MX_1.75u_PCB -> Button_Switch_Keyboard:SW_Cherry_MX_1.00u_PCB
- SW64, SW68: footprint Button_Switch_Keyboard:SW_Cherry_MX_2.25u_PCB -> Button_Switch_Keyboard:SW_Cherry_MX_1.00u_PCB
- SW66: footprint Button_Switch_Keyboard:SW_Cherry_MX_2.00u_PCB -> Button_Switch_Keyboard:SW_Cherry_MX_1.00u_PCB
- moved D60 374.6 mm to (471.2, 263.1)
- moved D36 359.9 mm to (462.6, 263.1)
- moved D63 353.5 mm to (475.5, 236.6)
- moved D64 345.7 mm to (475.5, 239.5)
- moved D62 342.9 mm to (456.3, 186.6)
- moved D65 336.1 mm to (475.5, 242.4)
- moved D49 327.2 mm to (103.7, 132.2)
- moved D40 308.0 mm to (466.9, 239.5)
- moved SW60 305.4 mm to (121.6, 109.2)
- moved D41 292.9 mm to (466.9, 242.4)
- moved SW36 291.4 mm to (426.4, 147.3)
- moved D52 289.5 mm to (471.2, 239.5)
- moved SW24 286.7 mm to (402.6, 109.2)
- moved D42 278.8 mm to (466.9, 245.4)
- moved D37 275.0 mm to (99.4, 132.2)
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Connections:
- D1 pad 1: Net-(D1-K) -> Row0
- D1 pad 2: Pin8 -> Net-(D1-A)
- D10 pad 1: Net-(D10-K) -> Row3
- D10 pad 2: Pin8 -> Net-(D10-A)
- D11 pad 1: Net-(D11-K) -> Row4
- D11 pad 2: Pin8 -> Net-(D11-A)
- D12 pad 1: Net-(D12-K) -> Row5
- D12 pad 2: Pin8 -> Net-(D12-A)
- D13 pad 1: Net-(D13-K) -> Row0
- D13 pad 2: Pin10 -> Net-(D13-A)
- D14 pad 1: Net-(D14-K) -> Row1
- D14 pad 2: Pin10 -> Net-(D14-A)
- D15 pad 1: Net-(D15-K) -> Row2
- D15 pad 2: Pin10 -> Net-(D15-A)
- D16 pad 1: Net-(D16-K) -> Row3
- D16 pad 2: Pin10 -> Net-(D16-A)
- D17 pad 1: Net-(D17-K) -> Row4
- D17 pad 2: Pin10 -> Net-(D17-A)
- D18 pad 1: Net-(D18-K) -> Row5
- D18 pad 2: Pin10 -> Net-(D18-A)
- D19 pad 1: Net-(D19-K) -> Row0
- D19 pad 2: Pin10 -> Net-(D19-A)
- D2 pad 1: Net-(D2-K) -> Row1
- D2 pad 2: Pin8 -> Net-(D2-A)
- D20 pad 1: Net-(D20-K) -> Row1
- D20 pad 2: Pin10 -> Net-(D20-A)
- D21 pad 1: Net-(D21-K) -> Row2
- D21 pad 2: Pin10 -> Net-(D21-A)
- D22 pad 1: Net-(D22-K) -> Row3
- D22 pad 2: Pin10 -> Net-(D22-A)
- D23 pad 1: Net-(D23-K) -> Row4
- D23 pad 2: Pin10 -> Net-(D23-A)
- D24 pad 1: Net-(D24-K) -> Row5
- D24 pad 2: Pin10 -> Net-(D24-A)
- D25 pad 1: Net-(D132-K) -> Row0
- D25 pad 2: Pin12 -> Net-(D25-A)
- D26 pad 1: Net-(D121-K) -> Row1
- D26 pad 2: Pin12 -> Net-(D26-A)
- D27 pad 1: Net-(D122-K) -> Row2
- D27 pad 2: Pin12 -> Net-(D27-A)
- D28 pad 1: Net-(D123-K) -> Row3
- D28 pad 2: Pin12 -> Net-(D28-A)
- D29 pad 1: Net-(D124-K) -> Row4
- D29 pad 2: Pin12 -> Net-(D29-A)
- D3 pad 1: Net-(D3-K) -> Row2
- D3 pad 2: Pin8 -> Net-(D3-A)
- D30 pad 1: Net-(D125-K) -> Row5
- D30 pad 2: Pin12 -> Net-(D30-A)
- D31 pad 1: Net-(D126-K) -> Row0
- D31 pad 2: Pin12 -> Net-(D31-A)
- D32 pad 1: Net-(D127-K) -> Row1
- D32 pad 2: Pin12 -> Net-(D32-A)
- D33 pad 1: Net-(D128-K) -> Row2
- D33 pad 2: Pin12 -> Net-(D33-A)
- D34 pad 1: Net-(D129-K) -> Row3
- D34 pad 2: Pin12 -> Net-(D34-A)
- D35 pad 1: Net-(D130-K) -> Row4
- D35 pad 2: Pin12 -> Net-(D35-A)
- D36 pad 1: Net-(D131-K) -> Row5
- D36 pad 2: Pin12 -> Net-(D36-A)
- D37 pad 1: Net-(D108-K) -> Row0
- D37 pad 2: Pin9 -> Net-(D37-A)
- D38 pad 1: Net-(D38-K) -> Row1
- D38 pad 2: Pin9 -> Net-(D38-A)
- D39 pad 1: Net-(D39-K) -> Row2
- D39 pad 2: Pin9 -> Net-(D39-A)
- D4 pad 1: Net-(D4-K) -> Row3
- D4 pad 2: Pin8 -> Net-(D4-A)
- D40 pad 1: Net-(D40-K) -> Row3
- D40 pad 2: Pin9 -> Net-(D40-A)
- D41 pad 1: Net-(D100-K) -> Row4
- D41 pad 2: Pin9 -> Net-(D41-A)
- D42 pad 1: Net-(D101-K) -> Row5
- D42 pad 2: Pin9 -> Net-(D42-A)
- D43 pad 1: Net-(D102-K) -> Row0
- D43 pad 2: Pin9 -> Net-(D43-A)
- D44 pad 1: Net-(D103-K) -> Row1
- D44 pad 2: Pin9 -> Net-(D44-A)
- D45 pad 1: Net-(D104-K) -> Row2
- D45 pad 2: Pin9 -> Net-(D45-A)
- D46 pad 1: Net-(D105-K) -> Row3
- D46 pad 2: Pin9 -> Net-(D46-A)
- D47 pad 1: Net-(D106-K) -> Row4
- D47 pad 2: Pin9 -> Net-(D47-A)
- D48 pad 1: Net-(D107-K) -> Row5
- D48 pad 2: Pin9 -> Net-(D48-A)
- D49 pad 1: Net-(D120-K) -> Row0
- D49 pad 2: Pin11 -> Net-(D49-A)
- D5 pad 1: Net-(D5-K) -> Row4
- D5 pad 2: Pin8 -> Net-(D5-A)
- D50 pad 1: Net-(D109-K) -> Row1
- D50 pad 2: Pin11 -> Net-(D50-A)
- D51 pad 1: Net-(D110-K) -> Row2
- D51 pad 2: Pin11 -> Net-(D51-A)
- D52 pad 1: Net-(D111-K) -> Row3
- D52 pad 2: Pin11 -> Net-(D52-A)
- D53 pad 1: Net-(D112-K) -> Row4
- D53 pad 2: Pin11 -> Net-(D53-A)
- D54 pad 1: Net-(D113-K) -> Row5
- D54 pad 2: Pin11 -> Net-(D54-A)
- D55 pad 1: Net-(D114-K) -> Row0
- D55 pad 2: Pin11 -> Net-(D55-A)
- D56 pad 1: Net-(D115-K) -> Row1
- D56 pad 2: Pin11 -> Net-(D56-A)
- D57 pad 1: Net-(D116-K) -> Row2
- D57 pad 2: Pin11 -> Net-(D57-A)
- D58 pad 1: Net-(D117-K) -> Row3
- D58 pad 2: Pin11 -> Net-(D58-A)
- D59 pad 1: Net-(D118-K) -> Row4
- D59 pad 2: Pin11 -> Net-(D59-A)
- D6 pad 1: Net-(D6-K) -> Row5
- D6 pad 2: Pin8 -> Net-(D6-A)
- D60 pad 1: Net-(D119-K) -> Row5
- D60 pad 2: Pin11 -> Net-(D60-A)
- D61 pad 1: Net-(D144-K) -> Row0
- D61 pad 2: Pin7 -> Net-(D61-A)
- D62 pad 1: Net-(D133-K) -> Row1
- D62 pad 2: Pin7 -> Net-(D62-A)
- D63 pad 1: Net-(D134-K) -> Row2
- D63 pad 2: Pin7 -> Net-(D63-A)
- D64 pad 1: Net-(D135-K) -> Row3
- D64 pad 2: Pin7 -> Net-(D64-A)
- D65 pad 1: Net-(D136-K) -> Row4
- D65 pad 2: Pin7 -> Net-(D65-A)
- D66 pad 1: Net-(D137-K) -> Row5
- D66 pad 2: Pin7 -> Net-(D66-A)
- D67 pad 1: Net-(D138-K) -> Row0
- D67 pad 2: Pin7 -> Net-(D67-A)
- D68 pad 1: Net-(D139-K) -> Row1
- D68 pad 2: Pin7 -> Net-(D68-A)
- D69 pad 1: Net-(D140-K) -> Row2
- D69 pad 2: Pin7 -> Net-(D69-A)
- D7 pad 1: Net-(D7-K) -> Row0
- D7 pad 2: Pin8 -> Net-(D7-A)
- D70 pad 1: Net-(D141-K) -> Row3
- D70 pad 2: Pin7 -> Net-(D70-A)
- D71 pad 1: Net-(D142-K) -> Row4
- D71 pad 2: Pin7 -> Net-(D71-A)
- D72 pad 1: Net-(D143-K) -> Row5
- D72 pad 2: Pin7 -> Net-(D72-A)
- D8 pad 1: Net-(D8-K) -> Row1
- D8 pad 2: Pin8 -> Net-(D8-A)
- D9 pad 1: Net-(D9-K) -> Row2
- D9 pad 2: Pin8 -> Net-(D9-A)
- J1 pad 1: Col12 -> Row1
- J1 pad 10: Pin10 -> Col1
- J1 pad 11: Pin11 -> Col2
- J1 pad 12: Pin12 -> Col3
- J1 pad 2: Col11 -> Row0
- J1 pad 5: Col10 -> Row2
- J1 pad 6: Col9 -> Row3
- J1 pad 7: Pin7 -> Row4
- J1 pad 8: Pin8 -> Row5
- J1 pad 9: Pin9 -> Col0
- J2 pad 1: Col1 -> Col4
- J2 pad 2: Col2 -> Col5
- J2 pad 3: Col3 -> Col6
- J2 pad 4: Col4 -> Col7
- J2 pad 5: Col5 -> Col8
- J2 pad 6: Col6 -> Col9
- J2 pad 7: Col7 -> Col10
- J2 pad 8: Col8 -> Col11
- SW1 pad 1: Net-(D1-K) -> Col0
- SW1 pad 2: GND -> Net-(D1-A)
- SW10 pad 1: Net-(D10-K) -> Col1
- SW10 pad 2: GND -> Net-(D10-A)
- SW11 pad 1: Net-(D11-K) -> Col1
- SW11 pad 2: GND -> Net-(D11-A)
- SW12 pad 1: Net-(D12-K) -> Col1
- SW12 pad 2: GND -> Net-(D12-A)
- SW13 pad 1: Net-(D14-K) -> Col2
- SW13 pad 2: GND -> Net-(D13-A)
- SW14 pad 1: Net-(D15-K) -> Col2
- SW14 pad 2: GND -> Net-(D14-A)
- SW15 pad 1: Net-(D16-K) -> Col2
- SW15 pad 2: GND -> Net-(D15-A)
- SW16 pad 1: Net-(D17-K) -> Col2
- SW16 pad 2: GND -> Net-(D16-A)
- SW17 pad 1: Net-(D18-K) -> Col2
- SW17 pad 2: GND -> Net-(D17-A)
- SW18 pad 1: Net-(D19-K) -> Col2
- SW18 pad 2: GND -> Net-(D18-A)
- SW19 pad 1: Net-(D20-K) -> Col3
- SW19 pad 2: GND -> Net-(D19-A)
- SW2 pad 1: Net-(D2-K) -> Col0
- SW2 pad 2: GND -> Net-(D2-A)
- SW20 pad 1: Net-(D21-K) -> Col3
- SW20 pad 2: GND -> Net-(D20-A)
- SW21 pad 1: Net-(D22-K) -> Col3
- SW21 pad 2: GND -> Net-(D21-A)
- SW22 pad 1: Net-(D23-K) -> Col3
- SW22 pad 2: GND -> Net-(D22-A)
- SW23 pad 1: Net-(D24-K) -> Col3
- SW23 pad 2: GND -> Net-(D23-A)
- SW24 pad 1: Net-(D13-K) -> Col3
- SW24 pad 2: GND -> Net-(D24-A)
- SW25 pad 1: Net-(D121-K) -> Col4
- SW25 pad 2: GND -> Net-(D25-A)
- SW26 pad 1: Net-(D122-K) -> Col4
- SW26 pad 2: GND -> Net-(D26-A)
- SW27 pad 1: Net-(D123-K) -> Col4
- SW27 pad 2: GND -> Net-(D27-A)
- SW28 pad 1: Net-(D124-K) -> Col4
- SW28 pad 2: GND -> Net-(D28-A)
- SW29 pad 1: Net-(D125-K) -> Col4
- SW29 pad 2: GND -> Net-(D29-A)
- SW3 pad 1: Net-(D3-K) -> Col0
- SW3 pad 2: GND -> Net-(D3-A)
- SW30 pad 1: Net-(D126-K) -> Col4
- SW30 pad 2: GND -> Net-(D30-A)
- SW31 pad 1: Net-(D127-K) -> Col5
- SW31 pad 2: GND -> Net-(D31-A)
- SW32 pad 1: Net-(D128-K) -> Col5
- SW32 pad 2: GND -> Net-(D32-A)
- SW33 pad 1: Net-(D129-K) -> Col5
- SW33 pad 2: GND -> Net-(D33-A)
- SW34 pad 1: Net-(D130-K) -> Col5
- SW34 pad 2: GND -> Net-(D34-A)
- SW35 pad 1: Net-(D131-K) -> Col5
- SW35 pad 2: GND -> Net-(D35-A)
- SW36 pad 1: Net-(D132-K) -> Col5
- SW36 pad 2: GND -> Net-(D36-A)
- SW37 pad 1: Net-(D38-K) -> Col6
- SW37 pad 2: GND -> Net-(D37-A)
- SW38 pad 1: Net-(D39-K) -> Col6
- SW38 pad 2: GND -> Net-(D38-A)
- SW39 pad 1: Net-(D40-K) -> Col6
- SW39 pad 2: GND -> Net-(D39-A)
- SW4 pad 1: Net-(D4-K) -> Col0
- SW4 pad 2: GND -> Net-(D4-A)
- SW40 pad 1: Net-(D100-K) -> Col6
- SW40 pad 2: GND -> Net-(D40-A)
- SW41 pad 1: Net-(D101-K) -> Col6
- SW41 pad 2: GND -> Net-(D41-A)
- SW42 pad 1: Net-(D102-K) -> Col6
- SW42 pad 2: GND -> Net-(D42-A)
- SW43 pad 1: Net-(D103-K) -> Col7
- SW43 pad 2: GND -> Net-(D43-A)
- SW44 pad 1: Net-(D104-K) -> Col7
- SW44 pad 2: GND -> Net-(D44-A)
- SW45 pad 1: Net-(D105-K) -> Col7
- SW45 pad 2: GND -> Net-(D45-A)
- SW46 pad 1: Net-(D106-K) -> Col7
- SW46 pad 2: GND -> Net-(D46-A)
- SW47 pad 1: Net-(D107-K) -> Col7
- SW47 pad 2: GND -> Net-(D47-A)
- SW48 pad 1: Net-(D108-K) -> Col7
- SW48 pad 2: GND -> Net-(D48-A)
- SW49 pad 1: Net-(D109-K) -> Col8
- SW49 pad 2: GND -> Net-(D49-A)
- SW5 pad 1: Net-(D5-K) -> Col0
- SW5 pad 2: GND -> Net-(D5-A)
- SW50 pad 1: Net-(D110-K) -> Col8
- SW50 pad 2: GND -> Net-(D50-A)
- SW51 pad 1: Net-(D111-K) -> Col8
- SW51 pad 2: GND -> Net-(D51-A)
- SW52 pad 1: Net-(D112-K) -> Col8
- SW52 pad 2: GND -> Net-(D52-A)
- SW53 pad 1: Net-(D113-K) -> Col8
- SW53 pad 2: GND -> Net-(D53-A)
- SW54 pad 1: Net-(D114-K) -> Col8
- SW54 pad 2: GND -> Net-(D54-A)
- SW55 pad 1: Net-(D115-K) -> Col9
- SW55 pad 2: GND -> Net-(D55-A)
- SW56 pad 1: Net-(D116-K) -> Col9
- SW56 pad 2: GND -> Net-(D56-A)
- SW57 pad 1: Net-(D117-K) -> Col9
- SW57 pad 2: GND -> Net-(D57-A)
- SW58 pad 1: Net-(D118-K) -> Col9
- SW58 pad 2: GND -> Net-(D58-A)
- SW59 pad 1: Net-(D119-K) -> Col9
- SW59 pad 2: GND -> Net-(D59-A)
- SW6 pad 1: Net-(D6-K) -> Col0
- SW6 pad 2: GND -> Net-(D6-A)
- SW60 pad 1: Net-(D120-K) -> Col9
- SW60 pad 2: GND -> Net-(D60-A)
- SW61 pad 1: Net-(D133-K) -> Col10
- SW61 pad 2: GND -> Net-(D61-A)
- SW62 pad 1: Net-(D134-K) -> Col10
- SW62 pad 2: GND -> Net-(D62-A)
- SW63 pad 1: Net-(D135-K) -> Col10
- SW63 pad 2: GND -> Net-(D63-A)
- SW64 pad 1: Net-(D136-K) -> Col10
- SW64 pad 2: GND -> Net-(D64-A)
- SW65 pad 1: Net-(D137-K) -> Col10
- SW65 pad 2: GND -> Net-(D65-A)
- SW66 pad 1: Net-(D138-K) -> Col10
- SW66 pad 2: GND -> Net-(D66-A)
- SW67 pad 1: Net-(D139-K) -> Col11
- SW67 pad 2: GND -> Net-(D67-A)
- SW68 pad 1: Net-(D140-K) -> Col11
- SW68 pad 2: GND -> Net-(D68-A)
- SW69 pad 1: Net-(D141-K) -> Col11
- SW69 pad 2: GND -> Net-(D69-A)
- SW7 pad 1: Net-(D7-K) -> Col1
- SW7 pad 2: GND -> Net-(D7-A)
- SW70 pad 1: Net-(D142-K) -> Col11
- SW70 pad 2: GND -> Net-(D70-A)
- SW71 pad 1: Net-(D143-K) -> Col11
- SW71 pad 2: GND -> Net-(D71-A)
- SW72 pad 1: Net-(D144-K) -> Col11
- SW72 pad 2: GND -> Net-(D72-A)
- SW8 pad 1: Net-(D8-K) -> Col1
- SW8 pad 2: GND -> Net-(D8-A)
- SW9 pad 1: Net-(D9-K) -> Col1
- SW9 pad 2: GND -> Net-(D9-A)
Routing:
- net Col12: track 593.0 -> 0.00 mm, vias 9 -> 0
- net Pin7: track 536.0 -> 0.00 mm, vias 12 -> 0
- net Pin11: track 530.0 -> 0.00 mm, vias 14 -> 0
- net Col11: track 511.8 -> 0.00 mm, vias 9 -> 0
- net Pin12: track 413.1 -> 0.00 mm, vias 15 -> 0
- net Col5: track 405.7 -> 0.00 mm, vias 10 -> 0
- net Pin10: track 362.4 -> 0.00 mm, vias 14 -> 0
- net Col6: track 340.5 -> 0.00 mm, vias 9 -> 0
- net Col1: track 334.1 -> 0.00 mm, vias 8 -> 0
- net Col4: track 305.1 -> 0.00 mm, vias 6 -> 0
- net Col2: track 300.9 -> 0.00 mm, vias 6 -> 0
- net Col3: track 295.3 -> 0.00 mm, vias 5 -> 0
- net Col7: track 292.6 -> 0.00 mm, vias 7 -> 0
- net Col10: track 283.2 -> 0.00 mm, vias 8 -> 0
- net Col8: track 263.1 -> 0.00 mm, vias 6 -> 0
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- removed copper zone on B.Cu, net (none)
Other:
- board text removed: "Michael Hollmer Custom Keyboard Design v1.0"

Commit message: Fixed matrix design
Parts:
- moved D60 390.6 mm to (113.6, 106.0)
- moved D29 368.3 mm to (113.6, 125.1)
- moved D18 359.3 mm to (113.6, 144.1)
- moved D6 350.2 mm to (113.6, 163.2)
- moved D7 342.7 mm to (151.7, 87.0)
- moved D8 326.7 mm to (161.4, 106.0)
- moved D4 323.8 mm to (144.6, 144.1)
- moved D5 318.2 mm to (145.8, 163.2)
- moved D9 315.5 mm to (166.2, 125.1)
- moved D19 313.3 mm to (189.8, 87.0)
- moved D10 300.6 mm to (175.5, 144.1)
- moved D11 300.4 mm to (169.7, 163.2)
- moved D20 296.9 mm to (199.4, 106.0)
- moved D17 286.8 mm to (182.7, 163.2)
- moved D21 285.3 mm to (204.0, 125.1)
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Routing:
- net Row4: track 0.00 -> 598.5 mm, vias 0 -> 12
- net Row5: track 0.00 -> 578.4 mm, vias 0 -> 14
- net Col4: track 0.00 -> 465.6 mm, vias 0 -> 2
- net Col1: track 0.00 -> 368.2 mm, vias 0 -> 4
- net Col3: track 0.00 -> 353.6 mm, vias 0 -> 3
- net Col9: track 0.00 -> 341.1 mm, vias 0 -> 2
- net Row3: track 0.00 -> 335.0 mm, vias 0 -> 13
- net Col5: track 0.00 -> 317.3 mm, vias 0 -> 3
- net Col0: track 0.00 -> 303.7 mm, vias 0 -> 1
- net Row2: track 0.00 -> 302.6 mm, vias 0 -> 12
- net Row1: track 0.00 -> 292.6 mm, vias 0 -> 14
- net Col6: track 0.00 -> 282.0 mm, vias 0 -> 4
- net Col2: track 0.00 -> 273.9 mm, vias 0 -> 2
- net Col10: track 0.00 -> 265.4 mm, vias 0 -> 3
- net Row0: track 0.00 -> 262.2 mm, vias 0 -> 13
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- added copper zone on B.Cu, net (none)
Other:
- board size 326.4 x 132.1 mm -> 326.4 x 133.3 mm
- board text added: "Michael Hollmer Custom Keyboard Design v.1.1"

Commit message: Final production layout
Routing:
- net Row5: track 578.4 -> 575.6 mm
Changed lines of the file:
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@@
     (property "ki_keywords" "connector")
     (attr through_hole)
-    (fp_text reference "J1" (at 0 -2.33) (layer "F.SilkS")
+    (fp_text reference "J1" (at -1.016 30.48) (layer "F.SilkS")
         (effects (font (size 1 1) (thickness 0.15)))
     )
@@
   (via (at 391.9855 106.045) (size 0.8) (drill 0.4) (layers "F.Cu" "B.Cu") (free) (net 26))
   (via (at 368.1095 106.045) (size 0.8) (drill 0.4) (layers "F.Cu" "B.Cu") (net 26))
-  (segment (start 244.4115 84.963) (end 247.2055 84.963) (width 0.25) (layer "B.Cu") (net 26))
   (segment (start 368.1095 106.045) (end 391.9855 106.045) (width 0.25) (layer "B.Cu") (net 26))
   (segment (start 260.6675 72.009) (end 260.9215 71.755) (width 0.25) (layer "B.Cu") (net 26))

Commit message: Started layout
Parts:
- removed D66, D72: D, Diode_SMD:D_SOD-323
- removed SW66, SW72: SW_Push, Button_Switch_Keyboard:SW_Cherry_MX_1.00u_PCB
- added C1: 0.1uF, Capacitor_SMD:C_0402_1005Metric, F.Cu at (259.4, 222.2)
- added C2: 1uF, Capacitor_SMD:C_0603_1608Metric, F.Cu at (282.8, 210.8)
- added D100: LED, LED_SMD:LED_0402_1005Metric, F.Cu at (195.2, 121.9)
- added D101: LED, LED_SMD:LED_0402_1005Metric, F.Cu at (223.9, 121.9)
- added D102: LED, LED_SMD:LED_0402_1005Metric, F.Cu at (243.0, 121.9)
- added D103: LED, LED_SMD:LED_0402_1005Metric, F.Cu at (262.0, 121.9)
- added D104: LED, LED_SMD:LED_0402_1005Metric, F.Cu at (281.1, 121.9)
- added D105: LED, LED_SMD:LED_0402_1005Metric, F.Cu at (309.3, 121.9)
- added D106: LED, LED_SMD:LED_0402_1005Metric, F.Cu at (328.6, 121.9)
- added D107: LED, LED_SMD:LED_0402_1005Metric, F.Cu at (347.6, 121.9)
- added D108: LED, LED_SMD:LED_0402_1005Metric, F.Cu at (366.7, 121.9)
- added D109: LED, LED_SMD:LED_0402_1005Metric, F.Cu at (395.4, 121.9)
- added D110: LED, LED_SMD:LED_0402_1005Metric, F.Cu at (423.8, 121.9)
- added D113: LED, LED_SMD:LED_0402_1005Metric, F.Cu at (128.7, 150.6)
- added D114: LED, LED_SMD:LED_0402_1005Metric, F.Cu at (147.8, 150.6)
- added D115: LED, LED_SMD:LED_0402_1005Metric, F.Cu at (166.6, 150.6)
- added D116: LED, LED_SMD:LED_0402_1005Metric, F.Cu at (185.6, 150.6)
- added D117: LED, LED_SMD:LED_0402_1005Metric, F.Cu at (204.6, 150.6)
- added D118: LED, LED_SMD:LED_0402_1005Metric, F.Cu at (223.9, 150.6)
- added D119: LED, LED_SMD:LED_0402_1005Metric, F.Cu at (242.7, 150.6)
- added D120: LED, LED_SMD:LED_0402_1005Metric, F.Cu at (262.0, 150.6)
- added D121: LED, LED_SMD:LED_0402_1005Metric, F.Cu at (281.1, 150.6)
- added D122: LED, LED_SMD:LED_0402_1005Metric, F.Cu at (300.1, 150.6)
- added D123: LED, LED_SMD:LED_0402_1005Metric, F.Cu at (319.2, 150.6)
- added D124: LED, LED_SMD:LED_0402_1005Metric, F.Cu at (338.2, 150.6)
- added D125: LED, LED_SMD:LED_0402_1005Metric, F.Cu at (357.3, 150.6)
- added D126: LED, LED_SMD:LED_0402_1005Metric, F.Cu at (386.0, 150.6)
- added D127: LED, LED_SMD:LED_0402_1005Metric, F.Cu at (423.8, 150.6)
- added D129: LED, LED_SMD:LED_0402_1005Metric, F.Cu at (133.5, 169.7)
- added D130: LED, LED_SMD:LED_0402_1005Metric, F.Cu at (157.1, 169.7)
- added D131: LED, LED_SMD:LED_0402_1005Metric, F.Cu at (176.4, 169.7)
- added D132: LED, LED_SMD:LED_0402_1005Metric, F.Cu at (195.2, 169.7)
- added D133: LED, LED_SMD:LED_0402_1005Metric, F.Cu at (214.3, 169.7)
- added D134: LED, LED_SMD:LED_0402_1005Metric, F.Cu at (233.3, 169.7)
- added D135: LED, LED_SMD:LED_0402_1005Metric, F.Cu at (252.6, 169.7)
- added D136: LED, LED_SMD:LED_0402_1005Metric, F.Cu at (271.4, 169.7)
- added D137: LED, LED_SMD:LED_0402_1005Metric, F.Cu at (290.7, 169.7)
- added D138: LED, LED_SMD:LED_0402_1005Metric, F.Cu at (309.5, 169.7)
- added D139: LED, LED_SMD:LED_0402_1005Metric, F.Cu at (328.6, 169.7)
- added D140: LED, LED_SMD:LED_0402_1005Metric, F.Cu at (347.6, 169.7)
- added D141: LED, LED_SMD:LED_0402_1005Metric, F.Cu at (366.7, 169.7)
- added D142: LED, LED_SMD:LED_0402_1005Metric, F.Cu at (390.8, 169.7)
- added D143: LED, LED_SMD:LED_0402_1005Metric, F.Cu at (423.8, 169.7)
- added D145: LED, LED_SMD:LED_0402_1005Metric, F.Cu at (135.8, 188.7)
- added D146: LED, LED_SMD:LED_0402_1005Metric, F.Cu at (162.0, 188.7)
- added D147: LED, LED_SMD:LED_0402_1005Metric, F.Cu at (181.3, 188.7)
- added D148: LED, LED_SMD:LED_0402_1005Metric, F.Cu at (200.1, 188.7)
- added D149: LED, LED_SMD:LED_0402_1005Metric, F.Cu at (219.1, 188.7)
- added D150: LED, LED_SMD:LED_0402_1005Metric, F.Cu at (238.4, 188.7)
- added D151: LED, LED_SMD:LED_0402_1005Metric, F.Cu at (257.2, 188.7)
- added D152: LED, LED_SMD:LED_0402_1005Metric, F.Cu at (276.3, 188.7)
- added D153: LED, LED_SMD:LED_0402_1005Metric, F.Cu at (295.3, 188.7)
- added D154: LED, LED_SMD:LED_0402_1005Metric, F.Cu at (314.4, 188.7)
- added D155: LED, LED_SMD:LED_0402_1005Metric, F.Cu at (333.4, 188.7)
- added D156: LED, LED_SMD:LED_0402_1005Metric, F.Cu at (352.5, 188.7)
- added D157: LED, LED_SMD:LED_0402_1005Metric, F.Cu at (383.5, 188.7)
- added D158: LED, LED_SMD:LED_0402_1005Metric, F.Cu at (423.8, 188.7)
- added D161: LED, LED_SMD:LED_0402_1005Metric, F.Cu at (140.6, 207.8)
- added D162: LED, LED_SMD:LED_0402_1005Metric, F.Cu at (171.6, 207.8)
- added D163: LED, LED_SMD:LED_0402_1005Metric, F.Cu at (190.7, 207.8)
- added D164: LED, LED_SMD:LED_0402_1005Metric, F.Cu at (209.5, 207.8)
- added D165: LED, LED_SMD:LED_0402_1005Metric, F.Cu at (228.8, 207.8)
- added D166: LED, LED_SMD:LED_0402_1005Metric, F.Cu at (247.8, 207.8)
- added D167: LED, LED_SMD:LED_0402_1005Metric, F.Cu at (266.9, 207.8)
- added D168: LED, LED_SMD:LED_0402_1005Metric, F.Cu at (285.9, 207.8)
- added D169: LED, LED_SMD:LED_0402_1005Metric, F.Cu at (305.0, 207.8)
- added D170: LED, LED_SMD:LED_0402_1005Metric, F.Cu at (324.0, 207.8)
- added D171: LED, LED_SMD:LED_0402_1005Metric, F.Cu at (343.1, 207.8)
- added D172: LED, LED_SMD:LED_0402_1005Metric, F.Cu at (369.2, 207.8)
- added D173: LED, LED_SMD:LED_0402_1005Metric, F.Cu at (405.0, 217.2)
- added D177: LED, LED_SMD:LED_0402_1005Metric, F.Cu at (131.0, 226.8)
- added D178: LED, LED_SMD:LED_0402_1005Metric, F.Cu at (154.9, 226.8)
- added D179: LED, LED_SMD:LED_0402_1005Metric, F.Cu at (178.7, 226.8)
- added D180: LED, LED_SMD:LED_0402_1005Metric, F.Cu at (250.1, 226.8)
- added D181: LED, LED_SMD:LED_0402_1005Metric, F.Cu at (319.2, 226.8)
- added D182: LED, LED_SMD:LED_0402_1005Metric, F.Cu at (338.5, 226.8)
- added D183: LED, LED_SMD:LED_0402_1005Metric, F.Cu at (357.3, 226.8)
- added D184: LED, LED_SMD:LED_0402_1005Metric, F.Cu at (385.7, 236.2)
- added D185: LED, LED_SMD:LED_0402_1005Metric, F.Cu at (405.0, 236.2)
- added D186: LED, LED_SMD:LED_0402_1005Metric, F.Cu at (423.8, 236.2)
- added D73: D, Diode_SMD:D_SOD-323, F.Cu at (389.9, 106.2)
- added D74: D, Diode_SMD:D_SOD-323, F.Cu at (351.8, 134.6)
- added D75: D, Diode_SMD:D_SOD-323, F.Cu at (361.4, 153.7)
- added D76: D, Diode_SMD:D_SOD-323, F.Cu at (378.2, 172.7)
- added D77: D, Diode_SMD:D_SOD-323, F.Cu at (399.5, 201.4)
- added D79: D, Diode_SMD:D_SOD-323, F.Cu at (418.8, 105.9)
- added D80: D, Diode_SMD:D_SOD-323, F.Cu at (380.7, 134.6)
- added D81: D, Diode_SMD:D_SOD-323, F.Cu at (385.3, 153.7)
- added D82: D, Diode_SMD:D_SOD-323, F.Cu at (418.6, 172.7)
- added D86: D, Diode_SMD:D_SOD-323, F.Cu at (418.3, 134.6)
- added D87: D, Diode_SMD:D_SOD-323, F.Cu at (418.6, 153.7)
- added D97: LED, LED_SMD:LED_0402_1005Metric, F.Cu at (128.7, 121.9)
- added D98: LED, LED_SMD:LED_0402_1005Metric, F.Cu at (157.4, 121.9)
- added D99: LED, LED_SMD:LED_0402_1005Metric, F.Cu at (176.2, 121.9)
- added InputC1: 100uF, Capacitor_SMD:C_1206_3216Metric, F.Cu at (347.7, 128.1)
- added J3: USB_VOLTAGE Measuring Point, Connector_PinHeader_2.54mm:PinHeader_1x01_P2.54mm_Vertical, F.Cu at (233.4, 120.0)
- added J4: LED_VOLTAGE Measuring Point 1, Connector_PinHeader_2.54mm:PinHeader_1x01_P2.54mm_Vertical, F.Cu at (271.5, 120.0)
- added J5: LED_VOLTAGE Measuring Point 2, Connector_PinHeader_2.54mm:PinHeader_1x01_P2.54mm_Vertical, F.Cu at (252.4, 120.0)
- added J6: Conn_01x02_Pin, Connector_PinHeader_2.54mm:PinHeader_1x02_P2.54mm_Vertical, F.Cu at (231.5, 217.2)
- added J7: Conn_01x02_Pin, Connector_PinHeader_2.54mm:PinHeader_1x02_P2.54mm_Vertical, F.Cu at (227.6, 217.2)
- added J8: Conn_01x02_Pin, Connector_PinHeader_2.54mm:PinHeader_1x02_P2.54mm_Vertical, F.Cu at (223.8, 217.2)
- added LEDPwr1: LED, LED_SMD:LED_0402_1005Metric, F.Cu at (261.5, 219.1)
- added LEDRPwr1: 65, Resistor_SMD:R_0201_0603Metric, F.Cu at (259.1, 219.1)
- added MicroUSB1: USB_OTG, Connector_USB:USB_Micro-B_Molex_47346-0001, F.Cu at (273.4, 96.6)
- added OutputC1: 100uF, Capacitor_SMD:C_1206_3216Metric, F.Cu at (332.4, 126.8)
- added Q1: IRLZ34N, Package_TO_SOT_SMD:TO-263-2, F.Cu at (141.9, 121.9)
- added Q2: IRLZ34N, Package_TO_SOT_SMD:TO-263-2, F.Cu at (380.7, 123.4)
- added Q3: IRLZ34N, Package_TO_SOT_SMD:TO-263-2, F.Cu at (407.4, 161.3)
- added Q4: IRLZ34N, Package_TO_SOT_SMD:TO-263-2, F.Cu at (409.7, 123.5)
- added Q5: IRLZ34N, Package_TO_SOT_SMD:TO-263-2, F.Cu at (209.2, 122.2)
- added Q6: IRLZ34N, Package_TO_SOT_SMD:TO-263-2, F.Cu at (295.4, 122.3)
- added R1: 10k, Resistor_SMD:R_0603_1608Metric, F.Cu at (230.4, 223.5)
- added R10: R, Resistor_SMD:R_0603_1608Metric, F.Cu at (258.8, 122.2)
- added R11: R, Resistor_SMD:R_0603_1608Metric, F.Cu at (278.4, 122.2)
- added R12: R, Resistor_SMD:R_0603_1608Metric, F.Cu at (306.2, 122.2)
- added R13: R, Resistor_SMD:R_0603_1608Metric, F.Cu at (325.9, 122.2)
- added R14: R, Resistor_SMD:R_0603_1608Metric, F.Cu at (344.7, 122.2)
- added R15: R, Resistor_SMD:R_0603_1608Metric, F.Cu at (363.7, 122.2)
- added R16: R, Resistor_SMD:R_0603_1608Metric, F.Cu at (392.4, 122.2)
- added R17: R, Resistor_SMD:R_0603_1608Metric, F.Cu at (420.9, 122.2)
- added R2: 10k, Resistor_SMD:R_0603_1608Metric, F.Cu at (261.5, 216.5)
- added R20: R, Resistor_SMD:R_0603_1608Metric, F.Cu at (125.5, 150.9)
- added R21: R, Resistor_SMD:R_0603_1608Metric, F.Cu at (144.8, 150.9)
- added R22: R, Resistor_SMD:R_0603_1608Metric, F.Cu at (163.6, 150.9)
- added R23: R, Resistor_SMD:R_0603_1608Metric, F.Cu at (201.2, 150.9)
- added R24: R, Resistor_SMD:R_0603_1608Metric, F.Cu at (220.9, 150.9)
- added R25: R, Resistor_SMD:R_0603_1608Metric, F.Cu at (239.5, 150.9)
- added R26: R, Resistor_SMD:R_0603_1608Metric, F.Cu at (259.1, 150.9)
- added R27: R, Resistor_SMD:R_0603_1608Metric, F.Cu at (277.9, 150.9)
- added R28: R, Resistor_SMD:R_0603_1608Metric, F.Cu at (296.9, 150.9)
- added R29: R, Resistor_SMD:R_0603_1608Metric, F.Cu at (316.0, 150.9)
- added R3: 10k, Resistor_SMD:R_0603_1608Metric, F.Cu at (225.9, 223.5)
- added R30: R, Resistor_SMD:R_0603_1608Metric, F.Cu at (335.0, 150.9)
- added R31: R, Resistor_SMD:R_0603_1608Metric, F.Cu at (354.1, 150.8)
- added R32: R, Resistor_SMD:R_0603_1608Metric, F.Cu at (382.5, 150.9)
- added R33: R, Resistor_SMD:R_0603_1608Metric, F.Cu at (420.4, 150.9)
- added R36: R, Resistor_SMD:R_0603_1608Metric, F.Cu at (129.8, 169.9)
- added R37: R, Resistor_SMD:R_0603_1608Metric, F.Cu at (153.4, 169.9)
- added R38: R, Resistor_SMD:R_0603_1608Metric, F.Cu at (173.0, 169.9)
- added R39: R, Resistor_SMD:R_0603_1608Metric, F.Cu at (191.8, 169.9)
- added R4: R, Resistor_SMD:R_0603_1608Metric, F.Cu at (125.7, 122.2)
- added R40: R, Resistor_SMD:R_0603_1608Metric, F.Cu at (210.8, 169.9)
- added R41: R, Resistor_SMD:R_0603_1608Metric, F.Cu at (229.9, 169.9)
- added R42: R, Resistor_SMD:R_0603_1608Metric, F.Cu at (249.4, 169.9)
- added R43: R, Resistor_SMD:R_0603_1608Metric, F.Cu at (268.2, 169.9)
- added R44: R, Resistor_SMD:R_0603_1608Metric, F.Cu at (287.3, 169.9)
- added R45: R, Resistor_SMD:R_0603_1608Metric, F.Cu at (306.1, 169.9)
- added R46: R, Resistor_SMD:R_0603_1608Metric, F.Cu at (324.9, 169.9)
- added R47: R, Resistor_SMD:R_0603_1608Metric, F.Cu at (344.4, 169.9)
- added R48: R, Resistor_SMD:R_0603_1608Metric, F.Cu at (363.2, 169.9)
- added R49: R, Resistor_SMD:R_0603_1608Metric, F.Cu at (387.3, 169.9)
- added R5: R, Resistor_SMD:R_0603_1608Metric, F.Cu at (154.4, 122.2)
- added R50: R, Resistor_SMD:R_0603_1608Metric, F.Cu at (419.9, 169.9)
- added R52: R, Resistor_SMD:R_0603_1608Metric, F.Cu at (132.6, 189.0)
- added R53: R, Resistor_SMD:R_0603_1608Metric, F.Cu at (158.5, 189.0)
- added R54: R, Resistor_SMD:R_0603_1608Metric, F.Cu at (177.5, 189.0)
- added R55: R, Resistor_SMD:R_0603_1608Metric, F.Cu at (196.6, 189.0)
- added R56: R, Resistor_SMD:R_0603_1608Metric, F.Cu at (215.4, 189.0)
- added R57: R, Resistor_SMD:R_0603_1608Metric, F.Cu at (234.9, 189.0)
- added R58: R, Resistor_SMD:R_0603_1608Metric, F.Cu at (253.2, 189.0)
- added R59: R, Resistor_SMD:R_0603_1608Metric, F.Cu at (272.8, 189.0)
- added R6: R, Resistor_SMD:R_0603_1608Metric, F.Cu at (173.2, 122.2)
- added R60: R, Resistor_SMD:R_0603_1608Metric, F.Cu at (291.8, 189.0)
- added R61: R, Resistor_SMD:R_0603_1608Metric, F.Cu at (310.6, 189.0)
- added R62: R, Resistor_SMD:R_0603_1608Metric, F.Cu at (329.9, 189.0)
- added R63: R, Resistor_SMD:R_0603_1608Metric, F.Cu at (349.0, 189.0)
- added R64: R, Resistor_SMD:R_0603_1608Metric, F.Cu at (380.0, 189.0)
- added R65: R, Resistor_SMD:R_0603_1608Metric, F.Cu at (420.9, 189.0)
- added R68: R, Resistor_SMD:R_0603_1608Metric, F.Cu at (137.7, 208.0)
- added R69: R, Resistor_SMD:R_0603_1608Metric, F.Cu at (168.4, 208.0)
- added R7: R, Resistor_SMD:R_0603_1608Metric, F.Cu at (192.5, 122.2)
- added R70: R, Resistor_SMD:R_0603_1608Metric, F.Cu at (186.9, 208.0)
- added R71: R, Resistor_SMD:R_0603_1608Metric, F.Cu at (206.0, 208.0)
- added R72: R, Resistor_SMD:R_0603_1608Metric, F.Cu at (225.0, 208.0)
- added R73: R, Resistor_SMD:R_0603_1608Metric, F.Cu at (244.1, 208.0)
- added R74: R, Resistor_SMD:R_0603_1608Metric, F.Cu at (262.9, 208.0)
- added R75: R, Resistor_SMD:R_0603_1608Metric, F.Cu at (281.7, 208.0)
- added R76: R, Resistor_SMD:R_0603_1608Metric, F.Cu at (301.5, 208.0)
- added R77: R, Resistor_SMD:R_0603_1608Metric, F.Cu at (320.8, 208.0)
- added R78: R, Resistor_SMD:R_0603_1608Metric, F.Cu at (339.6, 208.0)
- added R79: R, Resistor_SMD:R_0603_1608Metric, F.Cu at (365.5, 208.0)
- added R8: R, Resistor_SMD:R_0603_1608Metric, F.Cu at (221.2, 122.2)
- added R80: R, Resistor_SMD:R_0603_1608Metric, F.Cu at (401.8, 217.4)
- added R84: R, Resistor_SMD:R_0603_1608Metric, F.Cu at (127.0, 227.1)
- added R85: R, Resistor_SMD:R_0603_1608Metric, F.Cu at (150.9, 227.1)
- added R86: R, Resistor_SMD:R_0603_1608Metric, F.Cu at (175.0, 227.1)
- added R87: R, Resistor_SMD:R_0603_1608Metric, F.Cu at (246.4, 227.1)
- added R88: R, Resistor_SMD:R_0603_1608Metric, F.Cu at (315.7, 227.1)
- added R89: R, Resistor_SMD:R_0603_1608Metric, F.Cu at (334.5, 227.1)
- added R9: R, Resistor_SMD:R_0603_1608Metric, F.Cu at (240.0, 122.2)
- added R90: R, Resistor_SMD:R_0603_1608Metric, F.Cu at (353.8, 227.1)
- added R91: R, Resistor_SMD:R_0603_1608Metric, F.Cu at (382.0, 236.5)
- added R92: R, Resistor_SMD:R_0603_1608Metric, F.Cu at (401.2, 236.5)
- added R93: R, Resistor_SMD:R_0603_1608Metric, F.Cu at (420.3, 236.5)
- added SW76: SW_Push, Button_Switch_Keyboard:SW_Cherry_MX_1.00u_PCB, F.Cu at (397.8, 109.2)
- added SW77: SW_Push, Button_Switch_Keyboard:SW_Cherry_MX_1.00u_PCB, F.Cu at (359.7, 137.8)
- added SW78: SW_Push, Button_Switch_Keyboard:SW_Cherry_MX_1.00u_PCB, F.Cu at (369.3, 156.8)
- added SW79: SW_Push, Button_Switch_Keyboard:SW_Cherry_MX_2.25u_PCB, F.Cu at (385.9, 175.9)
- added SW80: SW_Push, Button_Switch_Keyboard:SW_Cherry_MX_1.00u_PCB, F.Cu at (407.4, 204.5)
- added SW82: SW_Push, Button_Switch_Keyboard:SW_Cherry_MX_1.00u_PCB, F.Cu at (426.4, 109.2)
- added SW83: SW_Push, Button_Switch_Keyboard:SW_Cherry_MX_2.00u_PCB, F.Cu at (388.3, 137.8)
- added SW84: SW_Push, Button_Switch_Keyboard:SW_Cherry_MX_1.50u_PCB, F.Cu at (393.1, 156.8)
- added SW85: SW_Push, Button_Switch_Keyboard:SW_Cherry_MX_1.00u_PCB, F.Cu at (426.4, 175.9)
- added SW89: SW_Push, Button_Switch_Keyboard:SW_Cherry_MX_1.00u_PCB, F.Cu at (426.1, 137.8)
- added SW90: SW_Push, Button_Switch_Keyboard:SW_Cherry_MX_1.00u_PCB, F.Cu at (426.4, 156.8)
- added U1: STM32F103VBTx, Package_QFP:LQFP-100_14x14mm_P0.5mm, F.Cu at (272.7, 218.4)
- added U2: AMS1117-3.3, Package_TO_SOT_SMD:SOT-223-3_TabPin2, F.Cu at (232.1, 128.3)
- added U3: CH340C, Package_SO:SOIC-16_3.9x9.9mm_P1.27mm, F.Cu at (290.5, 218.4)
- added U4: AMS1117-3.3, Package_TO_SOT_SMD:SOT-223-3_TabPin2, F.Cu at (262.6, 128.3)
- added UartC1: 0.1uF, Capacitor_SMD:C_0402_1005Metric, F.Cu at (290.4, 210.8)
- added VoltageReg1: AMS1117-3.3, Package_TO_SOT_SMD:SOT-223-3_TabPin2, F.Cu at (340.0, 128.3)
- J1, J2: value Conn_01x12_Socket -> Conn_01x04_Pin; footprint Connector_PinHeader_2.54mm:PinHeader_1x12_P2.54mm_Vertical -> Connector_PinHeader_2.54mm:PinHeader_1x04_P2.54mm_Vertical
- SW11, SW17: footprint Button_Switch_Keyboard:SW_Cherry_MX_1.25u_PCB -> Button_Switch_Keyboard:SW_Cherry_MX_1.00u_PCB
- SW12: footprint Button_Switch_Keyboard:SW_Cherry_MX_2.00u_PCB -> Button_Switch_Keyboard:SW_Cherry_MX_1.25u_PCB
- SW18, SW6: footprint Button_Switch_Keyboard:SW_Cherry_MX_1.00u_PCB -> Button_Switch_Keyboard:SW_Cherry_MX_1.25u_PCB
- SW2: footprint Button_Switch_Keyboard:SW_Cherry_MX_1.50u_PCB -> Button_Switch_Keyboard:SW_Cherry_MX_1.00u_PCB
- SW23: footprint Button_Switch_Keyboard:SW_Cherry_MX_2.25u_PCB -> Button_Switch_Keyboard:SW_Cherry_MX_1.00u_PCB
- SW24: footprint Button_Switch_Keyboard:SW_Cherry_MX_1.50u_PCB -> Button_Switch_Keyboard:SW_Cherry_MX_6.25u_PCB
- SW3: footprint Button_Switch_Keyboard:SW_Cherry_MX_1.75u_PCB -> Button_Switch_Keyboard:SW_Cherry_MX_1.50u_PCB
- SW35: footprint Button_Switch_Keyboard:SW_Cherry_MX_6.25u_PCB -> Button_Switch_Keyboard:SW_Cherry_MX_1.00u_PCB
- SW4: footprint Button_Switch_Keyboard:SW_Cherry_MX_2.25u_PCB -> Button_Switch_Keyboard:SW_Cherry_MX_1.75u_PCB
- SW5: footprint Button_Switch_Keyboard:SW_Cherry_MX_1.25u_PCB -> Button_Switch_Keyboard:SW_Cherry_MX_2.25u_PCB
- SW70: footprint Button_Switch_Keyboard:SW_Cherry_MX_1.75u_PCB -> Button_Switch_Keyboard:SW_Cherry_MX_1.00u_PCB
- SW71: footprint Button_Switch_Keyboard:SW_Cherry_MX_1.00u_PCB -> Button_Switch_Keyboard:SW_Cherry_MX_1.75u_PCB
- moved D60 325.6 mm to (418.6, 220.2)
- moved SW60 325.5 mm to (426.4, 223.5)
- moved SW12 270.5 mm to (157.3, 214.0)
- moved D12 261.2 mm to (160.0, 210.8), turned to 180 degrees
- moved H2 207.2 mm to (423.9, 128.3)
- moved D23 195.2 mm to (204.2, 191.8)
- moved SW23 195.1 mm to (212.1, 194.9)
- moved D24 183.1 mm to (244.6, 210.8)
- moved SW24 183.0 mm to (252.6, 214.0)
- moved SW41 179.0 mm to (269.2, 194.9)
- moved D41 178.9 mm to (261.3, 191.8)
- moved J1 168.3 mm to (214.3, 214.6)
- moved J2 145.8 mm to (219.4, 214.6), turned to 0 degrees
- moved H3 144.3 mm to (157.2, 200.0)
- moved D29 128.3 mm to (223.2, 191.8)
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Connections:
- J1 pad 1: Row1 -> I2C_SDA
- J1 pad 2: Row0 -> I2C_SCL
- J1 pad 4: GND -> 3.3V
- J2 pad 1: Col4 -> GND
- J2 pad 2: Col5 -> SWCLK
- J2 pad 3: Col6 -> SWDIO
- J2 pad 4: Col7 -> 3.3V
Routing:
- net Row4: track 598.5 -> 0.00 mm, vias 12 -> 0
- net Row5: track 575.6 -> 0.00 mm, vias 14 -> 0
- net Col4: track 465.6 -> 0.00 mm, vias 2 -> 0
- net Col1: track 368.2 -> 0.00 mm, vias 4 -> 0
- net Col3: track 353.6 -> 0.00 mm, vias 3 -> 0
- net Col9: track 341.1 -> 0.00 mm, vias 2 -> 0
- net Row3: track 335.0 -> 0.00 mm, vias 13 -> 0
- net Col5: track 317.3 -> 0.00 mm, vias 3 -> 0
- net Col0: track 303.7 -> 0.00 mm, vias 1 -> 0
- net Row2: track 302.6 -> 0.00 mm, vias 12 -> 0
- net Row1: track 292.6 -> 0.00 mm, vias 14 -> 0
- net Col6: track 282.0 -> 0.00 mm, vias 4 -> 0
- net Col2: track 273.9 -> 0.00 mm, vias 2 -> 0
- net Col10: track 265.4 -> 0.00 mm, vias 3 -> 0
- net Row0: track 262.2 -> 0.00 mm, vias 13 -> 0
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- added copper zone on B.Cu, net 3.3V
- removed copper zone on B.Cu, net (none)
- removed copper zone on B.Cu, net 5V
Other:
- board outline removed
- board text removed: "Michael Hollmer Custom Keyboard Design v.1.1"
